File: RV_main_pcb_ESP32/CAN_Interface.kicad_sch (KiCad schematic)
At the start: 16 parts, among them U3 MCP2515-xSO, U5 TJA1051T, Y1 Crystal

Commit message: assembly V1
Parts:
- C7, C8: value C -> 27pF
Changed lines of the file:
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@@
     (in_bom yes) (on_board yes)
     (property "Reference" "C8" (id 0) (at 95.25 90.17 90))
-    (property "Value" "C" (id 1) (at 97.79 96.52 90))
+    (property "Value" "27pF" (id 1) (at 97.79 96.52 90))
     (property "Footprint" "Capacitor_SMD:C_0603_1608Metric" (id 2) (at 99.06 93.0148 0)
       (effects (font (size 1.27 1.27)) hide)
@@
     (in_bom yes) (on_board yes)
     (property "Reference" "C7" (id 0) (at 95.25 80.01 90))
-    (property "Value" "C" (id 1) (at 97.79 86.36 90))
+    (property "Value" "27pF" (id 1) (at 97.79 86.36 90))
     (property "Footprint" "Capacitor_SMD:C_0603_1608Metric" (id 2) (at 99.06 82.8548 0)
       (effects (font (size 1.27 1.27)) hide)
