File: RV_main_pcb_ESP32/RV_main_pcb_ESP32.kicad_sch (KiCad schematic)
At the start: 11 parts, among them J1 Conn_01x15_Female, J2 Conn_01x15_Female, U1 TP5400

Commit message: drawio
Parts:
- removed C?: 100uF, Capacitor_SMD:C_1206_3216Metric, symbol Device:C
- removed C?: 10uF, Capacitor_SMD:C_1206_3216Metric, symbol Device:C
- removed D? (x2): LED, symbol Device:LED
- removed D?: D_Schottky, Diode_SMD:D_SMB, symbol Device:D_Schottky
- removed L?: L, Inductor_SMD:L_Taiyo-Yuden_NR-50xx_HandSoldering, symbol Device:L
- removed R?: 1k, Resistor_SMD:R_0603_1608Metric, symbol Device:R
- removed R?: 1.1k, Resistor_SMD:R_0603_1608Metric, symbol Device:R
- removed U1: TP5400, TP5400:ESOP8-NPTH-0.3mm, symbol TP5400:TP5400
- added U?: MPU-9250, Sensor_Motion:InvenSense_QFN-24_3x3mm_P0.4mm, symbol Sensor_Motion:MPU-9250

Commit message: schematics
Parts:
- removed J1, J2: Conn_01x15_Female, Connector_PinHeader_2.54mm:PinHeader_1x15_P2.54mm_Vertical, symbol Connector:Conn_01x15_Female
- added A1: Arduino_Nano_v2.x, Module:Arduino_Nano, symbol MCU_Module:Arduino_Nano_v2.x
- added H1, H2, H3, H4: MountingHole, MountingHole:MountingHole_3.2mm_M3_ISO7380, symbol Mechanical:MountingHole
- added J1: Conn_01x07_Female, Connector_PinHeader_2.54mm:PinHeader_1x06_P2.54mm_Vertical, symbol Connector:Conn_01x07_Female
- added J2: Conn_01x03_Female, Connector_PinHeader_2.54mm:PinHeader_1x03_P2.54mm_Vertical, symbol Connector:Conn_01x03_Female
- added U1: ESP32_DevKit_V1_DOIT, esp32_devkit_v1_doit:esp32_devkit_v1_doit, symbol esp32_devkit_v1_doit:ESP32_DevKit_V1_DOIT
- gave numbers to parts that had none: 1
Connections:
- net ESP32_VIN: now also U1.15 (VIN)
- net GND: now also J1.6 (Pin_6), U1.14 (GND), U1.17 (GND)
- new net CAN_CS: A1.13 (D10), J1.5 (Pin_5)
- new net CAN_HIGH: J2.1 (Pin_1)
- new net CAN_LOW: J2.3 (Pin_3)
- new net CAN_MISO: A1.15 (D12), J1.4 (Pin_4)
- new net CAN_MOSI: A1.14 (D11), J1.3 (Pin_3)
- new net CAN_SCK: A1.16 (D13), J1.2 (Pin_2)
- new net CAN_VCC: J1.7 (Pin_7)
- new net ESP32_3V3: U1.16 (3V3)
- no-connect marks 0 -> 2
Other:
- moved on the sheet: U2

Commit message: Hardware
Parts:
- removed U2: MPU-9250, Sensor_Motion:InvenSense_QFN-24_3x3mm_P0.4mm, symbol Sensor_Motion:MPU-9250
- added C1, C2: 100nF, Capacitor_SMD:C_0402_1005Metric, symbol Device:C
- added C3, C4, C6: 0.1uF, Capacitor_SMD:C_0805_2012Metric, symbol Device:C
- added C5: 0.1uF, Capacitor_SMD:C_0603_1608Metric, symbol Device:C
- added F1: Fuse, symbol Device:Fuse
- added F?: 0.5A, Fuse:Fuse_1206_3216Metric, symbol Device:Fuse
- added J3: Conn_01x02_Male, Connector_Molex:Molex_Micro-Fit_3.0_43650-0200_1x02_P3.00mm_Horizontal, symbol Connector:Conn_01x02_Male
- added J4: Conn_01x02_Male, TerminalBlock:TerminalBlock_bornier-2_P5.08mm, symbol Connector:Conn_01x02_Male
- added J5: Conn_02x03_Top_Bottom, Connector_Molex:Molex_Mini-Fit_Jr_5569-06A2_2x03_P4.20mm_Horizontal, symbol Connector_Generic:Conn_02x03_Top_Bottom
- added JP1: Jumper_2_Open, Connector_PinHeader_2.54mm:PinHeader_1x02_P2.54mm_Vertical, symbol Jumper:Jumper_2_Open
- added JP2, JP3: SolderJumper_2_Open, Jumper:SolderJumper-2_P1.3mm_Open_RoundedPad1.0x1.5mm, symbol Jumper:SolderJumper_2_Open
- added R1, R2, R3, R4, R5, R6: 0, Resistor_SMD:R_1206_3216Metric, symbol Device:R
- added R10, R11: 4,7k, Resistor_SMD:R_0603_1608Metric, symbol Device:R
- added R7: 0.01, Resistor_SMD:R_0805_2012Metric, symbol Device:R
- added R8, R9: 10, Resistor_SMD:R_0603_1608Metric, symbol Device:R
- added U2: LM1117-5, Package_TO_SOT_SMD:SOT-223, symbol Regulator_Linear:LM1117-3.3
- added U3: TXS0102DCT, Package_SO:SSOP-8_2.95x2.8mm_P0.65mm, symbol Logic_LevelTranslator:TXS0102DCT
- added U4: INA226, Package_SO:VSSOP-10_3x3mm_P0.5mm, symbol Analog_ADC:INA226
Connections:
- net CAN_HIGH: now also R5.1
- net CAN_LOW: now also R6.1
- net ESP32_3V3: now also C1.2, U3.3 (VCCA)
- net ESP32_VIN: now also F?.2
- net GND: now also C1.1, C2.2, C3.2, C4.1, C6.2, J4.2 (Pin_2), J5.1 (Pin_1), U2.1 (GND), U3.2 (GND), U4.1 (A1), U4.2 (A0), U4.7 (GND)
- net ESP-32_SDA_3.3V: now reaches U1.26 (IO21)
- net ESP-32_SDA_3.3V: now also R1.1
- net ESP-32_SCL_3.3V: now reaches U1.29 (IO22)
- net ESP-32_SCL_3.3V: now also R2.1
- net NANO_SDA_5V: now reaches A1.23 (A4)
- net NANO_SDA_5V: now also R3.2
- net NANO_SCL_5V: now reaches A1.24 (A5)
- net NANO_SCL_5V: now also R4.2
- net NANO_5V: now reaches A1.27 (+5V)
- net NANO_5V: now also C2.1, U3.7 (VCCB)
- net NANO_VIN: now reaches A1.30 (VIN)
- new net: R1.2, U3.5 (A1)
- new net: R4.1, U3.1 (B2)
- new net: R8.2, U4.10 (Vin+)
- new net: R3.1, U3.8 (B1)
- new net: F1.2, JP1.1 (A), JP2.1 (A)
- new net: F1.1, J4.1 (Pin_1), J5.4 (Pin_4)
- new net: J3.1 (Pin_1), R5.2
- new net: J3.2 (Pin_2), R6.2
- new net: R2.2, U3.4 (A2)
- new net: R9.1, U4.9 (Vin-)
- new net +12V: C3.1, C5.1, JP3.1 (A), R7.1, R9.2, U2.3 (VI)
- new net +3V3: C6.1, R10.2, R11.1, U4.6 (VS)
- new net +5V: C4.2, F?.1, U2.2 (VO)
- new net BATTERY: C5.2, JP1.2 (B), JP2.2 (B), JP3.2 (B), R7.2, R8.1
- new net SCK: R11.2, U4.5 (SCL)
- new net SD: R10.1, U4.4 (SDA)
Other:
- note added: "12V to 5V"
- note added: "Battery Voltage input"
- note added: "I2C Levelshifter"
- note added: "INA Current sensor"
- moved on the sheet: A1, H1, H2, H3, H4, J1, J2, U1

Commit message: update
Parts:
- removed JP1: Jumper_2_Open, Connector_PinHeader_2.54mm:PinHeader_1x02_P2.54mm_Vertical, symbol Jumper:Jumper_2_Open
- removed JP2: SolderJumper_2_Open, Jumper:SolderJumper-2_P1.3mm_Open_RoundedPad1.0x1.5mm, symbol Jumper:SolderJumper_2_Open
- added C7, C8: 0.1uF, Capacitor_SMD:C_0805_2012Metric, symbol Device:C
- added DNP1, DNP2, DNP3, DNP5, DNP6, DNP7, DNP8: DNP_small, symbol Fabian_Barth:DNP_small
- added DNP4: DNP_large, symbol Fabian_Barth:DNP_large
- added JP1: SolderJumper_2_Open, Jumper:SolderJumper-2_P1.3mm_Open_RoundedPad1.0x1.5mm, symbol Jumper:SolderJumper_2_Open
- added Q1: AO3400A, Package_TO_SOT_SMD:SOT-23, symbol Transistor_FET:AO3400A
- added Q2: AO3401A, Package_TO_SOT_SMD:SOT-23, symbol Transistor_FET:AO3401A
- added R12, R14, R16, R17: 0, Resistor_SMD:R_0805_2012Metric, symbol Device:R
- added R13, R15: 10k, Resistor_SMD:R_0805_2012Metric, symbol Device:R
- added R18: 2,5k, Resistor_SMD:R_0603_1608Metric, symbol Device:R
- added U5: LM1117-5, Package_TO_SOT_SMD:SOT-223, symbol Regulator_Linear:LM1117-3.3
- F1: value Fuse -> 10A
- R5, R6: footprint Resistor_SMD:R_1206_3216Metric -> Resistor_SMD:R_0603_1608Metric
- gave numbers to parts that had none: 1
Connections:
- net +3V3 is gone; now on net NANO_3V3: C6.1, R10.2, R11.1, U4.6 (VS)
- net +12V: now also Q2.2 (S), R18.2
- net +5V: now also R13.2
- net BATTERY: now also F1.2
- net CAN_VCC: now also R16.1
- net ESP32_VIN: now also C8.2, JP1.2 (B), R15.2, U5.2 (VO); no longer F2.2
- net GND: now also C7.2, C8.1, Q1.2 (S), R12.1, R14.1; no longer U2.1 (GND)
- net NANO_5V: now also F2.2, R16.2
- net NANO_D7: now reaches A1.10 (D7)
- net NANO_D7: now also R17.1
- net NANO_3V3: now reaches A1.17 (3V3)
- net NANO_VIN: no longer names the net of A1.30 (VIN)
- new net: Q1.1 (G), R17.2
- new net: R12.2, R13.1, U2.1 (GND)
- new net: Q1.3 (D), Q2.1 (G), R18.1
- new net: R14.2, R15.1, U5.1 (GND)
- new net ESP-32_12V: C7.1, JP1.1 (A), Q2.3 (D), U5.3 (VI)
Other:
- note added: "12V - 5V ESP-32"
- note added: "12V - 5V NANO"
- note added: "ESP-32 VCC MOSFET"
- note added: "ToDo: - Namen vom I2C vom INA anpassen - Insert Optocoppler"
- note removed: "12V to 5V"
- moved on the sheet: C3, C4, F2, U2

Commit message: update
Parts:
- removed J5: Conn_02x03_Top_Bottom, Connector_Molex:Molex_Mini-Fit_Jr_5569-06A2_2x03_P4.20mm_Horizontal, symbol Connector_Generic:Conn_02x03_Top_Bottom
- removed Q2: AO3401A, Package_TO_SOT_SMD:SOT-23, symbol Transistor_FET:AO3401A
- added C10: (no value), symbol Device:C
- added C9: 10uF, Capacitor_SMD:C_0603_1608Metric, symbol Device:C
- added D1: LED, symbol Device:LED
- added D2: (no value), symbol Device:LED
- added D3: 1N4148W, Diode_SMD:D_SOD-123, symbol Diode:1N4148W
- added D4: (no value), symbol Diode:1N4148W
- added F3: (no value), symbol Device:Fuse
- added F4: 10A, symbol Device:Fuse
- added H5: (no value), symbol Mechanical:MountingHole
- added H6, H7, H8: MountingHole, MountingHole:MountingHole_4.3mm_M4_DIN965, symbol Mechanical:MountingHole
- added J5: (no value), symbol Connector:Conn_01x01_Female
- added J6: (no value), symbol Connector:Conn_01x02_Male
- added K1: SANYOU_SRD_Form_C, Relay_THT:Relay_SPDT_SANYOU_SRD_Series_Form_C, symbol Relay:SANYOU_SRD_Form_C
- added K2: (no value), symbol Relay:SANYOU_SRD_Form_C
- added Q2: AO3400A, Package_TO_SOT_SMD:SOT-23, symbol Transistor_FET:AO3400A
- added R19: R, symbol Device:R
- added R20, R22: (no value), symbol Device:R
- added R21: 100, symbol Device:R
- J4: value Conn_01x02_Male -> (none); footprint TerminalBlock:TerminalBlock_bornier-2_P5.08mm -> (none)
- R17: value 0 -> 10k; footprint Resistor_SMD:R_0805_2012Metric -> (none)
- R18: value 2,5k -> 10k; footprint Resistor_SMD:R_0603_1608Metric -> (none)
Connections:
- net +12V: now also F3.2, F4.2; no longer R18.2
- net ESP-32_12V: now also K2.3
- net GND: now also R17.2, R18.2, C10.2, C9.2, J5.1 (Pin_1), J6.2 (Pin_2), Q2.2 (S)
- net NANO_5V: now also C10.1, C9.1, D3.1 (K), D4.1 (K), K1.5, K2.5, R19.1, R20.1
- net NANO_D7: now also R18.1, R22.1; no longer R17.1
- net at Q1.1 (G): now also R21.2; no longer R17.2
- net at Q1.3 (D): now also D1.1 (K), D3.2 (A), K1.2; no longer R18.1
- net NANO_D6: now reaches A1.9 (D6)
- net NANO_D6: now also R17.1, R21.1
- new net: F3.1, K1.1
- new net: J6.1 (Pin_1), K1.3
- new net: D1.2 (A), R19.2
- new net: Q2.1 (G), R22.2
- new net: F4.1, K2.1
- new net: D2.1 (K), D4.2 (A), K2.2, Q2.3 (D)
- new net: D2.2 (A), R20.2
Other:
- note added: "ESP-32 RELAY"
- note added: "Kofferraumklappe RELAY"
- note removed: "ESP-32 VCC MOSFET"
- moved on the sheet: C7, C8, JP1, R14, R15, U1, U5

Commit message: update
Parts:
- removed A1: Arduino_Nano_v2.x, Module:Arduino_Nano, symbol MCU_Module:Arduino_Nano_v2.x
- removed C1, C2: 100nF, Capacitor_SMD:C_0402_1005Metric, symbol Device:C
- removed C10: (no value), symbol Device:C
- removed C3, C4, C7, C8: 0.1uF, Capacitor_SMD:C_0805_2012Metric, symbol Device:C
- removed C9: 10uF, Capacitor_SMD:C_0603_1608Metric, symbol Device:C
- removed D1: LED, symbol Device:LED
- removed D2: (no value), symbol Device:LED
- removed D3: 1N4148W, Diode_SMD:D_SOD-123, symbol Diode:1N4148W
- removed D4: (no value), symbol Diode:1N4148W
- removed DNP1, DNP2, DNP3, DNP5, DNP6, DNP7, DNP8: DNP_small, symbol Fabian_Barth:DNP_small
- removed DNP4: DNP_large, symbol Fabian_Barth:DNP_large
- removed F4: 10A, symbol Device:Fuse
- removed H1, H2, H3, H4: MountingHole, MountingHole:MountingHole_3.2mm_M3_ISO7380, symbol Mechanical:MountingHole
- removed J1: Conn_01x07_Female, Connector_PinHeader_2.54mm:PinHeader_1x06_P2.54mm_Vertical, symbol Connector:Conn_01x07_Female
- removed JP1, JP3: SolderJumper_2_Open, Jumper:SolderJumper-2_P1.3mm_Open_RoundedPad1.0x1.5mm, symbol Jumper:SolderJumper_2_Open
- removed K1: SANYOU_SRD_Form_C, Relay_THT:Relay_SPDT_SANYOU_SRD_Series_Form_C, symbol Relay:SANYOU_SRD_Form_C
- removed K2: (no value), symbol Relay:SANYOU_SRD_Form_C
- removed Q1, Q2: AO3400A, Package_TO_SOT_SMD:SOT-23, symbol Transistor_FET:AO3400A
- removed R12, R14, R16: 0, Resistor_SMD:R_0805_2012Metric, symbol Device:R
- removed R13, R15: 10k, Resistor_SMD:R_0805_2012Metric, symbol Device:R
- removed R17, R18: 10k, symbol Device:R
- removed R19: R, symbol Device:R
- removed R2, R3, R4: 0, Resistor_SMD:R_1206_3216Metric, symbol Device:R
- removed R20, R22: (no value), symbol Device:R
- removed R21: 100, symbol Device:R
- removed R5, R6: 0, Resistor_SMD:R_0603_1608Metric, symbol Device:R
- removed U1: ESP32_DevKit_V1_DOIT, esp32_devkit_v1_doit:esp32_devkit_v1_doit, symbol esp32_devkit_v1_doit:ESP32_DevKit_V1_DOIT
- removed U2, U5: LM1117-5, Package_TO_SOT_SMD:SOT-223, symbol Regulator_Linear:LM1117-3.3
- removed U3: TXS0102DCT, Package_SO:SSOP-8_2.95x2.8mm_P0.65mm, symbol Logic_LevelTranslator:TXS0102DCT
- added J1: Conn_01x02_Male, Connector_Molex:Molex_Micro-Fit_3.0_43650-0200_1x02_P3.00mm_Horizontal, symbol Connector:Conn_01x02_Male
- added J7, J8, J9: Conn_01x02_Male, TerminalBlock:TerminalBlock_bornier-2_P5.08mm, symbol Connector:Conn_01x02_Male
- F1: footprint (none) -> custom_librarys:Flachsicherung
- F3: value (none) -> 1A; footprint (none) -> Fuse:Fuse_1206_3216Metric
- H5: value (none) -> MountingHole; footprint (none) -> MountingHole:MountingHole_3.2mm_M3
- H6, H7, H8: footprint MountingHole:MountingHole_4.3mm_M4_DIN965 -> MountingHole:MountingHole_3.2mm_M3
- J2: value Conn_01x03_Female -> Molex Micro-fit 3x1; footprint Connector_PinHeader_2.54mm:PinHeader_1x03_P2.54mm_Vertical -> Connector_Molex:Molex_Micro-Fit_3.0_43650-0300_1x03_P3.00mm_Horizontal
- J4, J6: value (none) -> Conn_01x02_Male; footprint (none) -> TerminalBlock:TerminalBlock_bornier-2_P5.08mm
- J5: value (none) -> Conn_01x01_Female; footprint (none) -> Connector:Banana_Jack_1Pin
- R1: footprint Resistor_SMD:R_1206_3216Metric -> Resistor_SMD:R_0805_2012Metric
Connections:
- net CAN_HIGH is gone; now on net NANO_5V: J2.1 (Pin_1)
- net +12V: no longer F3.2
- net ESP-32_SDA_3.3V: no longer R1.1
- net GND: now also J2.2 (Pin_2), J1.1 (Pin_1), J7.2 (Pin_2), J8.2 (Pin_2), J9.2 (Pin_2)
- net NANO_5V: now also R1.1
- net NANO_D6: now also J1.2 (Pin_2)
- net LM1117 fixed voltage1/VOUT: now reaches F3.1
- net Relay 10A2/NO: now reaches J6.1 (Pin_1)
- net CAN Interface/VCC: now reaches R1.2
- net CAN Interface/CAN_H: now reaches J3.1 (Pin_1)
- net CAN Interface/CAN_L: now reaches J3.2 (Pin_2)
- net +5V renamed LM1117 fixed voltage/VOUT
- net CAN_LOW renamed ESP32_WS2812B_status_LED_5V
- net NANO_3V3 renamed ESP32_VCC
- net ESP32_VCC: now also F3.2
- new net Relay 10A/NO: J9.1 (Pin_1)
- new net Relay 10A1/NO: J7.1 (Pin_1)
- new net Relay 10A3/NO: J8.1 (Pin_1)
- no-connect marks 2 -> 21
Other:
- added sheet CAN Interface (CAN_Interface.kicad_sch)
- added sheet ESP32 (ESP32.kicad_sch)
- added sheet LM1117 fixed voltage (LM1117_fixed.kicad_sch)
- added sheet LM1117 fixed voltage1 (LM1117_fixed.kicad_sch)
- added sheet NANO (NANO.kicad_sch)
- added sheet Relay 10A (Relay_10A.kicad_sch)
- added sheet Relay 10A1 (Relay_10A.kicad_sch)
- added sheet Relay 10A2 (Relay_10A.kicad_sch)
- added sheet Relay 10A3 (Relay_10A.kicad_sch)
- added sheet TXS0102_instance1 (TXS0102.kicad_sch)
- added sheet TXS0102_instance2 (TXS0102.kicad_sch)
- note added: "ToDo: - Namen vom I2C vom INA anpassen - Kofferraumklappe relay von ESP steuern lassen - I2C TXS Levelshifter Pull-up überprüfen"
- note added: "WLED_ESP8266_molex_microfit RELAY"
- note added: "WS2812b Levelshifter"
- note added: "Zigarettenanzünder 1"
- note added: "Zigarettenanzünder 2"
- note removed: "12V - 5V ESP-32"
- note removed: "12V - 5V NANO"
- note removed: "ESP-32 RELAY"
- note removed: "ToDo: - Namen vom I2C vom INA anpassen - Insert Optocoppler"
- moved on the sheet: C5, C6, J3, R10, R11, R7, R8, R9, U4

Commit message: update
Parts:
- added J12, J13: Conn_01x02_Male, Connector_Molex:Molex_Micro-Fit_3.0_43650-0200_1x02_P3.00mm_Horizontal, symbol Connector:Conn_01x02_Male
Connections:
- net GND: now also J12.1 (Pin_1), J13.1 (Pin_1)
- net LM1117 fixed voltage/VOUT renamed +5V
- new net ESP_SW1: J12.2 (Pin_2)
- new net ESP_SW2: J13.2 (Pin_2)
- no-connect marks 21 -> 19
Other:
- removed sheet LM1117 fixed voltage
- added sheet 5V 3A Buck (5V_buck.kicad_sch)
- note added: "Camping Mode selection"
- note added: "ESP32 switch input 1"
- note added: "ESP32 switch input 2"
- note added: "ToDo: - Namen vom I2C vom INA anpassen - I2C TXS Levelshifter Pull-up überprüfen"
- note removed: "ToDo: - Namen vom I2C vom INA anpassen - Kofferraumklappe relay von ESP steuern lassen - I2C TXS Levelshifter Pull-up überprüfen"
- moved on the sheet: F2

Commit message: assembly V1
Changed lines of the file:
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@@
-    )
-  )
-  (global_label "NANO_5V" (shape input) (at 185.42 36.83 180) (fields_autoplaced)
-    (effects (font (size 1.27 1.27)) (justify right))
-    (property "Intersheet References" "${INTERSHEET_REFS}" (id 0) (at 174.6612 36.9094 0)
-      (effects (font (size 1.27 1.27)) (justify right) hide)
     )
   )
@@
     )
   )
-  (global_label "NANO_5V" (shape input) (at 241.3 36.83 180) (fields_autoplaced)
-    (effects (font (size 1.27 1.27)) (justify right))
-    (property "Intersheet References" "${INTERSHEET_REFS}" (id 0) (at 230.5412 36.9094 0)
-      (effects (font (size 1.27 1.27)) (justify right) hide)
-    )
-  )
   (global_label "CAN_CS" (shape input) (at 119.38 48.26 180) (fields_autoplaced)
     (effects (font (size 1.27 1.27)) (justify right))
@@
     )
   )
-  (global_label "NANO_5V" (shape input) (at 185.42 64.77 180) (fields_autoplaced)
-    (effects (font (size 1.27 1.27)) (justify right))
-    (property "Intersheet References" "${INTERSHEET_REFS}" (id 0) (at 174.6612 64.8494 0)
-      (effects (font (size 1.27 1.27)) (justify right) hide)
-    )
-  )
   (global_label "ESP32_RELAY_1" (shape input) (at 64.77 29.21 0) (fields_autoplaced)
     (effects (font (size 1.27 1.27)) (justify left))
@@
     )
   )
-  (global_label "NANO_5V" (shape input) (at 241.3 64.77 180) (fields_autoplaced)
-    (effects (font (size 1.27 1.27)) (justify right))
-    (property "Intersheet References" "${INTERSHEET_REFS}" (id 0) (at 230.5412 64.8494 0)
-      (effects (font (size 1.27 1.27)) (justify right) hide)
-    )
-  )
   (global_label "NANO_5V" (shape input) (at 139.7 177.8 0) (fields_autoplaced)
     (effects (font (size 1.27 1.27)) (justify left))
@@
     (pin "2")
   )
+  (symbol (lib_id "power:+5V") (at 241.3 64.77 90) (unit 1)
+    (in_bom yes) (on_board yes)
+    (property "Reference" "#PWR?" (id 0) (at 245.11 64.77 0)
+      (effects (font (size 1.27 1.27)) hide)
+    )
+    (property "Value" "+5V" (id 1) (at 233.68 64.77 90)
+      (effects (font (size 1.27 1.27)) (justify right))
+    )
+    (property "Footprint" "" (id 2) (at 241.3 64.77 0)
+      (effects (font (size 1.27 1.27)) hide)
+    )
+    (property "Datasheet" "" (id 3) (at 241.3 64.77 0)
+      (effects (font (size 1.27 1.27)) hide)
+    )
+    (pin "1")
+  )
   (symbol (lib_id "power:+12V") (at 210.82 63.5 270) (unit 1)
     (in_bom yes) (on_board yes) (fields_autoplaced)
@@
     (pin "2")
   )
+  (symbol (lib_id "power:+5V") (at 185.42 36.83 90) (unit 1)
+    (in_bom yes) (on_board yes)
+    (property "Reference" "#PWR?" (id 0) (at 189.23 36.83 0)
+      (effects (font (size 1.27 1.27)) hide)
+    )
+    (property "Value" "+5V" (id 1) (at 177.8 36.83 90)
+      (effects (font (size 1.27 1.27)) (justify right))
+    )
+    (property "Footprint" "" (id 2) (at 185.42 36.83 0)
+      (effects (font (size 1.27 1.27)) hide)
+    )
+    (property "Datasheet" "" (id 3) (at 185.42 36.83 0)
+      (effects (font (size 1.27 1.27)) hide)
+    )
+    (pin "1")
+  )
   (symbol (lib_id "Device:R") (at 231.14 138.43 90) (unit 1)
     (in_bom yes) (on_board yes)
@@
     (pin "2")
   )
+  (symbol (lib_id "power:+5V") (at 185.42 64.77 90) (unit 1)
+    (in_bom yes) (on_board yes)
+    (property "Reference" "#PWR?" (id 0) (at 189.23 64.77 0)
+      (effects (font (size 1.27 1.27)) hide)
+    )
+    (property "Value" "+5V" (id 1) (at 177.8 64.77 90)
+      (effects (font (size 1.27 1.27)) (justify right))
+    )
+    (property "Footprint" "" (id 2) (at 185.42 64.77 0)
+      (effects (font (size 1.27 1.27)) hide)
+    )
+    (property "Datasheet" "" (id 3) (at 185.42 64.77 0)
+      (effects (font (size 1.27 1.27)) hide)
+    )
+    (pin "1")
+  )
   (symbol (lib_id "power:GND") (at 195.58 124.46 90) (unit 1)
     (in_bom yes) (on_board yes)
@@
     )
     (property "Datasheet" "" (id 3) (at 27.94 143.51 0)
+      (effects (font (size 1.27 1.27)) hide)
+    )
+    (pin "1")
+  )
+  (symbol (lib_id "power:+5V") (at 241.3 36.83 90) (unit 1)
+    (in_bom yes) (on_board yes)
+    (property "Reference" "#PWR?" (id 0) (at 245.11 36.83 0)
+      (effects (font (size 1.27 1.27)) hide)
+    )
+    (property "Value" "+5V" (id 1) (at 233.68 36.83 90)
+      (effects (font (size 1.27 1.27)) (justify right))
+    )
+    (property "Footprint" "" (id 2) (at 241.3 36.83 0)
+      (effects (font (size 1.27 1.27)) hide)
+    )
+    (property "Datasheet" "" (id 3) (at 241.3 36.83 0)
       (effects (font (size 1.27 1.27)) hide)
     )
@@
       (reference "#PWR0165") (unit 1) (value "GND") (footprint "")
     )
+    (path "/44af3bb8-bc54-4ef1-a89b-e92604c23bcf"
+      (reference "#PWR?") (unit 1) (value "+5V") (footprint "")
+    )
+    (path "/88f42f1f-5b79-4315-a039-7bbb84228026"
+      (reference "#PWR?") (unit 1) (value "+5V") (footprint "")
+    )
+    (path "/9785d738-29f1-4fa7-a80b-eb854a0a947b"
+      (reference "#PWR?") (unit 1) (value "+5V") (footprint "")
+    )
+    (path "/a61d0d9c-9add-4a2d-9c75-454f4a001e5c"
+      (reference "#PWR?") (unit 1) (value "+5V") (footprint "")
+    )
     (path "/d8af53df-2092-4965-8eba-00cf85442882/336d8791-6675-4891-bf89-17fc79d5c9dc"
       (reference "C1") (unit 1) (value "0.1uF") (footprint "Capacitor_SMD:C_0805_2012Metric")
@@
     )
     (path "/eb3822a0-347c-4e64-8d15-826d07122948/b6d9b54f-e2b9-4118-b394-cf9228672cad"
-      (reference "C7") (unit 1) (value "C") (footprint "Capacitor_SMD:C_0603_1608Metric")
+      (reference "C7") (unit 1) (value "27pF") (footprint "Capacitor_SMD:C_0603_1608Metric")
     )
     (path "/eb3822a0-347c-4e64-8d15-826d07122948/ada9d573-f470-4c42-b26d-933060c497aa"
-      (reference "C8") (unit 1) (value "C") (footprint "Capacitor_SMD:C_0603_1608Metric")
+      (reference "C8") (unit 1) (value "27pF") (footprint "Capacitor_SMD:C_0603_1608Metric")
     )
     (path "/eb3822a0-347c-4e64-8d15-826d07122948/bfbce513-9500-4c40-9548-1f17822aeea0"
@@
     )
     (path "/f88dfef8-8d41-455d-98b9-e505b0fe42a0/ce445e93-a415-45b7-a1f8-141c71c4db6e"
-      (reference "R13") (unit 1) (value "R") (footprint "Resistor_SMD:R_0603_1608Metric")
+      (reference "R13") (unit 1) (value "100") (footprint "Resistor_SMD:R_0603_1608Metric")
     )
     (path "/eb3822a0-347c-4e64-8d15-826d07122948/0ec9e4d1-b596-4f74-8b23-53bb4751fddb"
@@
     )
     (path "/4c4116a0-6b54-48d2-93c5-74eff3e4b8a4/ce445e93-a415-45b7-a1f8-141c71c4db6e"
-      (reference "R22") (unit 1) (value "R") (footprint "Resistor_SMD:R_0603_1608Metric")
+      (reference "R22") (unit 1) (value "100") (footprint "Resistor_SMD:R_0603_1608Metric")
     )
     (path "/4c4116a0-6b54-48d2-93c5-74eff3e4b8a4/c1208492-656a-49b3-8528-76a169d1432f"
@@
     )
     (path "/4f5a8807-77ff-483d-b06b-d4aed27415c4/ce445e93-a415-45b7-a1f8-141c71c4db6e"
-      (reference "R30") (unit 1) (value "R") (footprint "Resistor_SMD:R_0603_1608Metric")
+      (reference "R30") (unit 1) (value "100") (footprint "Resistor_SMD:R_0603_1608Metric")
     )
     (path "/4f5a8807-77ff-483d-b06b-d4aed27415c4/c1208492-656a-49b3-8528-76a169d1432f"
@@
     )
     (path "/a7e0698a-f05d-4f5b-820f-174aa5c88ddd/ce445e93-a415-45b7-a1f8-141c71c4db6e"
-      (reference "R41") (unit 1) (value "R") (footprint "Resistor_SMD:R_0603_1608Metric")
+      (reference "R41") (unit 1) (value "100") (footprint "Resistor_SMD:R_0603_1608Metric")
     )
     (path "/a7e0698a-f05d-4f5b-820f-174aa5c88ddd/c1208492-656a-49b3-8528-76a169d1432f"
