File: RV_main_pcb_ESP32/RV_main_pcb_ESP32.kicad_sch (KiCad schematic)
At the start: 27 parts, among them J1 Conn_01x02_Male, J12 Conn_01x02_Male, J13 Conn_01x02_Male, J2 Molex Micro-fit 3x1, J3 Conn_01x02_Male, J4 Conn_01x02_Male, J5 Conn_01x01_Female, J6 Conn_01x02_Male, J7 Conn_01x02_Male, J8 Conn_01x02_Male, J9 Conn_01x02_Male, U4 INA226

Commit message: Software initial upload
Other:
- added sheet changelog (changelog.kicad_sch)
- note added: "Kofferraumbeleuchtung unten"
- note added: "ToDo: - Namen vom I2C vom INA anpassen - I2C TXS Levelshifter Pull-up überprüfen - Footprint DC DC Spule anpassen - Footprint DC DC Diode anpassen - ESP32: Add button EN -> GND - ADD UART header Atmega328p - Add 100nF to CH340C 3V3 - GND - Swap RX and TX on CH340C - remove 0 ohm resistors on Levelshifter - remove 0 ohm resistor on CAN interface - increase cap to 0603 on levelshifter - increase pa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"
- note removed: "ToDo: - Namen vom I2C vom INA anpassen - I2C TXS Levelshifter Pull-up überprüfen"
- note removed: "WLED_ESP8266_molex_microfit RELAY"
Changed lines of the file:
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@@
 (kicad_sch (version 20211123) (generator eeschema)
   (paper "A4")
+  (title_block
+    (date "2022-05-22")
+    (rev "1")
+  )
   (junction (at 194.31 124.46) (diameter 0) (color 0 0 0 0)
   )
@@
     (effects (font (size 2 2)) (justify left bottom))
   )
-  (text "ToDo:\n- Namen vom I2C vom INA anpassen\n- I2C TXS Levelshifter Pull-up überprüfen\n"
-    (at 168.91 163.83 0)
+  (text "ToDo:\n- Namen vom I2C vom INA anpassen\n- I2C TXS Levelshifter Pull-up überprüfen\n- Footprint DC DC Spule anpassen\n- Footprint DC DC Diode anpassen\n- ESP32: Add button EN -> GND\n- ADD UART header Atmega328p\n- Add 100nF to CH340C 3V3 - GND\n- Swap RX and TX on CH340C\n- remove 0 ohm resistors on Levelshifter\n- remove 0 ohm resistor on CAN interface\n- increase cap to 0603 on levelshifter\n- increase pad size of fuse holder\n- add reverse polarity protection\n- add ESD and EMV protection\n\n"
+    (at 92.71 151.13 0)
     (effects (font (size 1.27 1.27)) (justify left bottom))
   )
@@
     (effects (font (size 2 2)) (justify left bottom))
   )
-  (text "WLED_ESP8266_molex_microfit RELAY" (at 227.33 57.15 0)
+  (text "Kofferraumbeleuchtung unten" (at 233.68 57.15 0)
     (effects (font (size 1.8 1.8)) (justify left bottom))
   )
@@
     (pin "+5V" input (at 186.69 64.77 180)
       (effects (font (size 1.27 1.27)) (justify left))
+    )
+  )
+  (sheet (at 190.5 153.67) (size 25.4 11.43)
+    (stroke (width 0.1524) (type solid) (color 0 0 0 0))
+    (fill (color 0 0 0 0.0000))
+    (property "Sheet name" "changelog" (id 0) (at 198.12 156.21 0)
+      (effects (font (size 1.27 1.27)) (justify left bottom))
+    )
+    (property "Sheet file" "changelog.kicad_sch" (id 1) (at 190.5 162.56 0)
+      (effects (font (size 1.27 1.27)) (justify left top))
     )
   )
@@
     (path "/7cb6d2b6-7b36-4c3c-9606-c80baed356b5" (page "11"))
     (path "/a7e0698a-f05d-4f5b-820f-174aa5c88ddd" (page "12"))
+    (path "/b0b067cc-ca57-40a3-a560-afa57094e1fd" (page "13"))
     (path "/004c30d9-3726-4058-8db0-bb836a778fc7" (page "13"))
   )
