File: RV_main_pcb_ESP32/ESP32.kicad_sch (KiCad schematic)
At the start: 14 parts, among them J11 Conn_01x04_Male, Q1 AO3400A, Q4 AO3400A, SW2 SW_Push, U8 ESP32-WROOM-32

Commit message: Software initial upload
Other:
- note added: "Programming procedure: 1. USB to TTL wiring: TX - RX RX - TX GND - GND 2. HOLD FLASH continuously 3. Pull down EN short 4. Upload code (ESP32 DEVKIT V1) 5. After upload: release FLASH button 6. Pull down EN short to start board"
Changed lines of the file:
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@@
     (stroke (width 0) (type default) (color 0 0 0 0))
+  )
+  (text "Programming procedure:\n1. USB to TTL wiring:\n	TX - RX\n	RX - TX\n	GND - GND\n2. HOLD FLASH continuously\n3. Pull down EN short\n4. Upload code (ESP32 DEVKIT V1)\n5. After upload: release FLASH button\n6. Pull down EN short to start board\n"
+    (at 220.98 50.8 0)
+    (effects (font (size 2 2)) (justify left bottom))
   )
   (label "ESP_TX" (at 123.19 58.42 0)
