File: RV_main_pcb_ESP32/Relay_10A.kicad_sch (KiCad schematic)
At the start: 9 parts, among them K4 SANYOU_SRD_Form_C, Q6 AO3400A

Commit message: assembly V1
Parts:
- R41: value R -> 100
Changed lines of the file:
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@@
       (effects (font (size 1.27 1.27)) (justify left))
     )
-    (property "Value" "R" (id 1) (at 133.35 82.5499 0)
+    (property "Value" "100" (id 1) (at 133.35 82.5499 0)
       (effects (font (size 1.27 1.27)) (justify left))
     )

Commit message: Software initial upload
Parts:
- renumbered C28 to C11, D10 to D5, D11 to D6, F8 to F5, K4 to K3, Q6 to Q3, R40 to R20, R41 to R22, R42 to R23
Changed lines of the file:
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@@
   (symbol (lib_id "Transistor_FET:AO3400A") (at 146.05 105.41 0)
     (in_bom yes) (on_board yes)
-    (property "Reference" "Q6" (id 0) (at 151.13 102.87 0)
+    (property "Reference" "Q3" (id 0) (at 151.13 102.87 0)
       (effects (font (size 1.27 1.27)) (justify left))
     )
@@
   (symbol (lib_id "Device:C") (at 119.38 78.74 0)
     (in_bom yes) (on_board yes)
-    (property "Reference" "C28" (id 0) (at 121.92 77.47 0)
+    (property "Reference" "C11" (id 0) (at 121.92 77.47 0)
       (effects (font (size 1.27 1.27)) (justify left))
     )
@@
   (symbol (lib_id "Diode:1N4148W") (at 138.43 86.36 270)
     (in_bom yes) (on_board yes)
-    (property "Reference" "D11" (id 0) (at 133.35 86.36 90)
+    (property "Reference" "D6" (id 0) (at 133.35 86.36 90)
       (effects (font (size 1.27 1.27)) (justify left))
     )
@@
   (symbol (lib_id "power:GND") (at 119.38 83.82 0)
     (in_bom yes) (on_board yes)
-    (property "Reference" "#PWR0162" (id 0) (at 119.38 90.17 0)
+    (property "Reference" "#PWR0129" (id 0) (at 119.38 90.17 0)
       (effects (font (size 1.27 1.27)) hide)
     )
@@
   (symbol (lib_id "Device:Fuse") (at 162.56 101.6 90)
     (in_bom yes) (on_board yes)
-    (property "Reference" "F8" (id 0) (at 162.56 99.06 90))
+    (property "Reference" "F5" (id 0) (at 162.56 99.06 90))
     (property "Value" "10A" (id 1) (at 162.56 104.14 90))
     (property "Footprint" "custom_librarys:Flachsicherung" (id 2) (at 162.56 103.378 90)
@@
   (symbol (lib_id "Device:R") (at 134.62 105.41 90)
     (in_bom yes) (on_board yes)
-    (property "Reference" "R42" (id 0) (at 133.35 102.87 90))
+    (property "Reference" "R23" (id 0) (at 133.35 102.87 90))
     (property "Value" "100" (id 1) (at 134.62 107.95 90))
     (property "Footprint" "Resistor_SMD:R_0603_1608Metric" (id 2) (at 134.62 107.188 90)
@@
   (symbol (lib_id "Device:R") (at 127 109.22 0)
     (in_bom yes) (on_board yes)
-    (property "Reference" "R40" (id 0) (at 121.92 107.95 0)
+    (property "Reference" "R20" (id 0) (at 121.92 107.95 0)
       (effects (font (size 1.27 1.27)) (justify left))
     )
@@
   (symbol (lib_id "Device:LED") (at 130.81 91.44 90)
     (in_bom yes) (on_board yes) (fields_autoplaced)
-    (property "Reference" "D10" (id 0) (at 134.62 91.7574 90)
+    (property "Reference" "D5" (id 0) (at 134.62 91.7574 90)
       (effects (font (size 1.27 1.27)) (justify right))
     )
@@
   (symbol (lib_id "Relay:SANYOU_SRD_Form_C") (at 153.67 86.36 0)
     (in_bom yes) (on_board yes)
-    (property "Reference" "K4" (id 0) (at 165.1 85.0899 0)
+    (property "Reference" "K3" (id 0) (at 165.1 85.0899 0)
       (effects (font (size 1.27 1.27)) (justify left))
     )
@@
   (symbol (lib_id "Device:R") (at 130.81 81.28 0)
     (in_bom yes) (on_board yes) (fields_autoplaced)
-    (property "Reference" "R41" (id 0) (at 133.35 80.0099 0)
+    (property "Reference" "R22" (id 0) (at 133.35 80.0099 0)
       (effects (font (size 1.27 1.27)) (justify left))
     )
@@
   (symbol (lib_id "power:GND") (at 148.59 111.76 0)
     (in_bom yes) (on_board yes)
-    (property "Reference" "#PWR0160" (id 0) (at 148.59 118.11 0)
+    (property "Reference" "#PWR0127" (id 0) (at 148.59 118.11 0)
       (effects (font (size 1.27 1.27)) hide)
     )
@@
   (symbol (lib_id "power:GND") (at 127 114.3 0)
     (in_bom yes) (on_board yes)
-    (property "Reference" "#PWR0161" (id 0) (at 127 120.65 0)
+    (property "Reference" "#PWR0128" (id 0) (at 127 120.65 0)
       (effects (font (size 1.27 1.27)) hide)
     )
