File: RV_main_pcb_ESP32/RV_main_pcb_ESP32.kicad_pcb (KiCad board)
At the start: 2 copper layers, 1 part, among them U1 TP5400

Commit message: schematics
Parts:
- added A1: Arduino_Nano_v2.x, Module:Arduino_Nano, F.Cu at (130.5, 59.5)
- added H1: MountingHole, MountingHole:MountingHole_3.2mm_M3_ISO7380, F.Cu at (237.8, 150.9)
- added H2: MountingHole, MountingHole:MountingHole_3.2mm_M3_ISO7380, F.Cu at (242.4, 143.3)
- added H3: MountingHole, MountingHole:MountingHole_3.2mm_M3_ISO7380, F.Cu at (247.1, 133.6)
- added H4: MountingHole, MountingHole:MountingHole_3.2mm_M3_ISO7380, F.Cu at (247.3, 154.7)
- added J1: Conn_01x07_Female, Connector_PinHeader_2.54mm:PinHeader_1x06_P2.54mm_Vertical, F.Cu at (216.1, 134.9)
- added J2: Conn_01x03_Female, Connector_PinHeader_2.54mm:PinHeader_1x03_P2.54mm_Vertical, F.Cu at (241.1, 132.3)
- added U2: MPU-9250, Sensor_Motion:InvenSense_QFN-24_3x3mm_P0.4mm, F.Cu at (98.4, 109.9)
- U1: value TP5400 -> ESP32_DevKit_V1_DOIT; footprint TP5400:ESOP8-NPTH-0.3mm -> esp32_devkit_v1_doit:esp32_devkit_v1_doit
- moved U1 82.9 mm to (75.5, 46.1)

Commit message: Hardware
Parts:
- added C1: 100nF, Capacitor_SMD:C_0402_1005Metric, F.Cu at (77.8, 148.1)
- added C2: 100nF, Capacitor_SMD:C_0402_1005Metric, F.Cu at (74.9, 148.1)
- added C3: 0.1uF, Capacitor_SMD:C_0805_2012Metric, F.Cu at (30.5, 180.6)
- added C4: 0.1uF, Capacitor_SMD:C_0805_2012Metric, F.Cu at (46.4, 170.1)
- added C5: 0.1uF, Capacitor_SMD:C_0603_1608Metric, F.Cu at (50.6, 169.8)
- added C6: 0.1uF, Capacitor_SMD:C_0805_2012Metric, F.Cu at (35.0, 180.6)
- added J3: Conn_01x02_Male, Connector_Molex:Molex_Micro-Fit_3.0_43650-0200_1x02_P3.00mm_Horizontal, F.Cu at (61.9, 134.9)
- added J4: Conn_01x02_Male, TerminalBlock:TerminalBlock_bornier-2_P5.08mm, F.Cu at (49.6, 113.7)
- added J5: Conn_02x03_Top_Bottom, Connector_Molex:Molex_Mini-Fit_Jr_5569-06A2_2x03_P4.20mm_Horizontal, F.Cu at (32.0, 170.7)
- added JP1: Jumper_2_Open, Connector_PinHeader_2.54mm:PinHeader_1x02_P2.54mm_Vertical, F.Cu at (56.3, 158.1)
- added JP2: SolderJumper_2_Open, Jumper:SolderJumper-2_P1.3mm_Open_RoundedPad1.0x1.5mm, F.Cu at (46.3, 173.4)
- added JP3: SolderJumper_2_Open, Jumper:SolderJumper-2_P1.3mm_Open_RoundedPad1.0x1.5mm, F.Cu at (60.8, 157.6)
- added R1: 0, Resistor_SMD:R_1206_3216Metric, F.Cu at (88.0, 141.2)
- added R10: 4,7k, Resistor_SMD:R_0603_1608Metric, F.Cu at (39.2, 180.3)
- added R11: 4,7k, Resistor_SMD:R_0603_1608Metric, F.Cu at (58.0, 164.2)
- added R2: 0, Resistor_SMD:R_1206_3216Metric, F.Cu at (93.6, 141.2)
- added R3: 0, Resistor_SMD:R_1206_3216Metric, F.Cu at (88.0, 144.4)
- added R4: 0, Resistor_SMD:R_1206_3216Metric, F.Cu at (94.5, 136.8)
- added R5: 0, Resistor_SMD:R_1206_3216Metric, F.Cu at (33.3, 134.1)
- added R6: 0, Resistor_SMD:R_1206_3216Metric, F.Cu at (49.2, 119.9)
- added R7: 0.01, Resistor_SMD:R_0805_2012Metric, F.Cu at (53.7, 165.5)
- added R8: 10, Resistor_SMD:R_0603_1608Metric, F.Cu at (60.6, 160.6)
- added R9: 10, Resistor_SMD:R_0603_1608Metric, F.Cu at (50.6, 172.4)
- added U3: TXS0102DCT, Package_SO:SSOP-8_2.95x2.8mm_P0.65mm, F.Cu at (88.5, 137.3)
- added U4: INA226, Package_SO:VSSOP-10_3x3mm_P0.5mm, F.Cu at (47.8, 166.3)
- U2: value MPU-9250 -> LM1117-5; footprint Sensor_Motion:InvenSense_QFN-24_3x3mm_P0.4mm -> Package_TO_SOT_SMD:SOT-223
- moved U2 70.3 mm to (49.0, 159.9)
Connections:
- A1 pad 23: unconnected-(A1-Pad23) -> NANO_SDA_5V
- A1 pad 24: unconnected-(A1-Pad24) -> NANO_SCL_5V
- A1 pad 27: unconnected-(A1-Pad27) -> NANO_5V
- U1 pad 26: unconnected-(U1-Pad26) -> ESP-32_SDA_3.3V
- U1 pad 29: unconnected-(U1-Pad29) -> ESP-32_SCL_3.3V
- U2 pad 1: unconnected-(U2-Pad1) -> GND
- U2 pad 2: (no net) -> +5V
- U2 pad 3: (no net) -> +12V

Commit message: update
Parts:
- added C10: 10uF, Capacitor_SMD:C_0603_1608Metric, F.Cu at (210.4, 84.6)
- added C7: 0.1uF, Capacitor_SMD:C_0805_2012Metric, F.Cu at (213.4, 76.2)
- added C8: 0.1uF, Capacitor_SMD:C_0805_2012Metric, F.Cu at (219.1, 72.8)
- added C9: 10uF, Capacitor_SMD:C_0603_1608Metric, F.Cu at (213.1, 79.0)
- added D3: 1N4148W, Diode_SMD:D_SOD-123, F.Cu at (192.4, 93.8)
- added D4: 1N4148W, Diode_SMD:D_SOD-123, F.Cu at (214.0, 73.0)
- added F2: 0.5A, Fuse:Fuse_1206_3216Metric, F.Cu at (225.5, 63.9)
- added H5: MountingHole, MountingHole:MountingHole_4.3mm_M4_DIN965, F.Cu at (194.1, 87.6)
- added H6: MountingHole, MountingHole:MountingHole_4.3mm_M4_DIN965, F.Cu at (218.2, 66.8)
- added H7: MountingHole, MountingHole:MountingHole_4.3mm_M4_DIN965, F.Cu at (203.9, 84.9)
- added H8: MountingHole, MountingHole:MountingHole_4.3mm_M4_DIN965, F.Cu at (206.6, 75.9)
- added J5: Conn_01x01_Female, Connector:Banana_Jack_1Pin, F.Cu at (147.3, 160.0)
- added J6: Conn_01x02_Male, TerminalBlock:TerminalBlock_bornier-2_P5.08mm, F.Cu at (205.3, 66.8)
- added JP1: SolderJumper_2_Open, Jumper:SolderJumper-2_P1.3mm_Open_RoundedPad1.0x1.5mm, F.Cu at (230.5, 64.1)
- added K1: SANYOU_SRD_Form_C, Relay_THT:Relay_SPDT_SANYOU_SRD_Series_Form_C, F.Cu at (170.5, 70.8)
- added K2: SANYOU_SRD_Form_C, Relay_THT:Relay_SPDT_SANYOU_SRD_Series_Form_C, F.Cu at (170.5, 87.7)
- added Q1: AO3400A, Package_TO_SOT_SMD:SOT-23, F.Cu at (201.0, 91.7)
- added Q2: AO3400A, Package_TO_SOT_SMD:SOT-23, F.Cu at (225.1, 67.8)
- added R12: 0, Resistor_SMD:R_0805_2012Metric, F.Cu at (191.7, 97.0)
- added R13: 10k, Resistor_SMD:R_0805_2012Metric, F.Cu at (210.6, 81.9)
- added R14: 0, Resistor_SMD:R_0805_2012Metric, F.Cu at (217.8, 76.2)
- added R15: 10k, Resistor_SMD:R_0805_2012Metric, F.Cu at (196.2, 97.0)
- added R16: 0, Resistor_SMD:R_0805_2012Metric, F.Cu at (200.6, 95.4)
- added U5: LM1117-5, Package_TO_SOT_SMD:SOT-223, F.Cu at (194.5, 79.0)
- J4: footprint TerminalBlock:TerminalBlock_bornier-2_P5.08mm -> MountingHole:MountingHole_4.3mm_M4_ISO14580_Pad_TopBottom
- R5, R6: footprint Resistor_SMD:R_1206_3216Metric -> Resistor_SMD:R_0603_1608Metric
- moved J4 2.28 mm to (50.8, 111.8)
Connections:
- A1 pad 10: unconnected-(A1-Pad10) -> NANO_D7
- A1 pad 17: unconnected-(A1-Pad17) -> NANO_3V3
- A1 pad 9: unconnected-(A1-Pad9) -> NANO_D6
- C6 pad 1: +3V3 -> NANO_3V3
- J4 pad 1: Net-(J4-Pad1) -> Net-(F1-Pad1)
- R10 pad 2: +3V3 -> NANO_3V3
- R11 pad 1: +3V3 -> NANO_3V3
- U2 pad 1: GND -> Net-(R12-Pad2)
- U4 pad 6: +3V3 -> NANO_3V3

Commit message: update
Parts:
- removed A1: Arduino_Nano_v2.x, Module:Arduino_Nano
- removed H1, H2, H3, H4: MountingHole, MountingHole:MountingHole_3.2mm_M3_ISO7380
- removed the J5 at (32.0, 170.7)
- removed the JP1 at (230.5, 64.1)
- removed the JP1 at (56.3, 158.1)
- removed JP2, JP3: SolderJumper_2_Open, Jumper:SolderJumper-2_P1.3mm_Open_RoundedPad1.0x1.5mm
- added C11: 10uF, Capacitor_SMD:C_0603_1608Metric, F.Cu at (126.7, 96.6)
- added C12: C, Capacitor_SMD:C_0603_1608Metric, F.Cu at (183.0, 88.5)
- added C13: 100nF, Capacitor_SMD:C_0603_1608Metric, F.Cu at (182.2, 99.5)
- added C14: 100nF, Capacitor_SMD:C_0603_1608Metric, F.Cu at (181.8, 98.0)
- added C15: 100nF, Capacitor_SMD:C_0603_1608Metric, F.Cu at (196.5, 101.0)
- added C16: 4,7uF 16V, Capacitor_SMD:C_1206_3216Metric, F.Cu at (182.2, 103.2)
- added C17: 100nF, Capacitor_SMD:C_0603_1608Metric, F.Cu at (207.0, 100.5)
- added C18: 100nF, Capacitor_SMD:C_0603_1608Metric, F.Cu at (189.9, 111.9)
- added C19: 0.1uF, Capacitor_SMD:C_0603_1608Metric, F.Cu at (146.8, 110.3)
- added C20: 100nF, Capacitor_SMD:C_0603_1608Metric, F.Cu at (146.8, 107.0)
- added C21: 22uF, Capacitor_SMD:C_0603_1608Metric, F.Cu at (148.5, 107.0)
- added C22: 0.1uF, Capacitor_SMD:C_0603_1608Metric, F.Cu at (160.2, 133.0)
- added C23: 10uF, Capacitor_SMD:C_0603_1608Metric, F.Cu at (87.7, 97.1)
- added C24: 100nF, Capacitor_SMD:C_0402_1005Metric, F.Cu at (157.5, 84.2)
- added C25: 100nF, Capacitor_SMD:C_0402_1005Metric, F.Cu at (157.5, 92.8)
- added C26: 100nF, Capacitor_SMD:C_0402_1005Metric, F.Cu at (184.2, 125.6)
- added C27: 100nF, Capacitor_SMD:C_0402_1005Metric, F.Cu at (184.2, 133.8)
- added C28: 10uF, Capacitor_SMD:C_0603_1608Metric, F.Cu at (68.9, 97.1)
- added D1: GREEN, LED_SMD:LED_0805_2012Metric_Pad1.15x1.40mm_HandSolder, F.Cu at (177.5, 103.2)
- added D10: LED, LED_SMD:LED_0805_2012Metric_Pad1.15x1.40mm_HandSolder, F.Cu at (74.2, 101.1)
- added D11: 1N4148W, Diode_SMD:D_SOD-123, F.Cu at (74.2, 97.1)
- added D2: LED, LED_SMD:LED_0805_2012Metric_Pad1.15x1.40mm_HandSolder, F.Cu at (112.9, 101.1)
- added D5: LED, LED_SMD:LED_0805_2012Metric_Pad1.15x1.40mm_HandSolder, F.Cu at (132.4, 101.1)
- added D6: 1N4148W, Diode_SMD:D_SOD-123, F.Cu at (132.2, 96.6)
- added D7: GREEN, LED_SMD:LED_0805_2012Metric_Pad1.15x1.40mm_HandSolder, F.Cu at (140.5, 108.8)
- added D8: LED, LED_SMD:LED_0805_2012Metric_Pad1.15x1.40mm_HandSolder, F.Cu at (93.4, 101.1)
- added D9: 1N4148W, Diode_SMD:D_SOD-123, F.Cu at (93.4, 97.1)
- added F1: 10A, custom_librarys:Flachsicherung, F.Cu at (173.5, 79.5)
- added F3: 1A, Fuse:Fuse_1206_3216Metric, F.Cu at (147.2, 134.0)
- added F4: 10A, custom_librarys:Flachsicherung, F.Cu at (105.9, 123.6)
- added F5: 10A, custom_librarys:Flachsicherung, F.Cu at (111.9, 123.6)
- added F6: 0.5A, Fuse:Fuse_1206_3216Metric, F.Cu at (204.8, 100.5)
- added F7: 10A, custom_librarys:Flachsicherung, F.Cu at (99.9, 123.6)
- added F8: 10A, custom_librarys:Flachsicherung, F.Cu at (93.9, 123.6)
- added J10: USB_B_Micro, Connector_USB:USB_Micro-B_Molex_47346-0001, F.Cu at (206.5, 125.0)
- added J11: Conn_01x04_Male, Connector_PinHeader_2.54mm:PinHeader_1x04_P2.54mm_Vertical, F.Cu at (176.5, 116.7)
- added J7: Conn_01x02_Male, TerminalBlock:TerminalBlock_bornier-2_P5.08mm, F.Cu at (119.4, 63.5)
- added J8: Conn_01x02_Male, TerminalBlock:TerminalBlock_bornier-2_P5.08mm, F.Cu at (82.1, 63.5)
- added J9: Conn_01x02_Male, TerminalBlock:TerminalBlock_bornier-2_P5.08mm, F.Cu at (107.0, 63.5)
- added JP1: Jumper_2_Open, Connector_PinHeader_2.54mm:PinHeader_1x02_P2.54mm_Vertical, F.Cu at (181.5, 112.0)
- added K3: SANYOU_SRD_Form_C, Relay_THT:Relay_SPDT_SANYOU_SRD_Series_Form_C, F.Cu at (131.7, 92.6)
- added K4: SANYOU_SRD_Form_C, Relay_THT:Relay_SPDT_SANYOU_SRD_Series_Form_C, F.Cu at (74.2, 92.6)
- added Q3: AO3400A, Package_TO_SOT_SMD:SOT-23, F.Cu at (138.4, 100.8)
- added Q4: AO3400A, Package_TO_SOT_SMD:SOT-23, F.Cu at (143.8, 112.3)
- added Q5: AO3400A, Package_TO_SOT_SMD:SOT-23, F.Cu at (99.9, 100.8)
- added Q6: AO3400A, Package_TO_SOT_SMD:SOT-23, F.Cu at (80.2, 100.8)
- added R17: 0, Resistor_SMD:R_0805_2012Metric, F.Cu at (184.2, 72.5)
- added R18: 100, Resistor_SMD:R_0603_1608Metric, F.Cu at (117.9, 104.8)
- added R19: 1k, Resistor_SMD:R_0603_1608Metric, F.Cu at (191.0, 108.2)
- added R20: 10k, Resistor_SMD:R_0603_1608Metric, F.Cu at (139.2, 104.8)
- added R21: 1k, Resistor_SMD:R_0603_1608Metric, F.Cu at (192.5, 108.2)
- added R22: R, Resistor_SMD:R_0603_1608Metric, F.Cu at (132.4, 104.9)
- added R23: 100, Resistor_SMD:R_0603_1608Metric, F.Cu at (137.4, 104.8)
- added R24: 250, Resistor_SMD:R_0603_1608Metric, F.Cu at (179.8, 103.2)
- added R25: 10k, Resistor_SMD:R_0603_1608Metric, F.Cu at (200.5, 128.6)
- added R26: 125, Resistor_SMD:R_0603_1608Metric, F.Cu at (140.5, 112.8)
- added R27: 10k, Resistor_SMD:R_0603_1608Metric, F.Cu at (145.0, 108.5)
- added R28: 10k, Resistor_SMD:R_0603_1608Metric, F.Cu at (160.2, 134.5)
- added R29: 10k, Resistor_SMD:R_0603_1608Metric, F.Cu at (100.7, 104.8)
- added R30: R, Resistor_SMD:R_0603_1608Metric, F.Cu at (93.4, 104.8)
- added R31: 100, Resistor_SMD:R_0603_1608Metric, F.Cu at (98.9, 104.8)
- added R32: 0, Resistor_SMD:R_1206_3216Metric, F.Cu at (152.0, 90.2)
- added R33: 0, Resistor_SMD:R_1206_3216Metric, F.Cu at (152.0, 87.2)
- added R34: 0, Resistor_SMD:R_1206_3216Metric, F.Cu at (163.2, 90.2)
- added R35: 0, Resistor_SMD:R_1206_3216Metric, F.Cu at (163.2, 87.2)
- added R36: 0, Resistor_SMD:R_1206_3216Metric, F.Cu at (178.9, 131.6)
- added R37: 0, Resistor_SMD:R_1206_3216Metric, F.Cu at (178.9, 128.1)
- added R38: 0, Resistor_SMD:R_1206_3216Metric, F.Cu at (190.2, 131.6)
- added R39: 0, Resistor_SMD:R_1206_3216Metric, F.Cu at (190.2, 128.1)
- added R40: 10k, Resistor_SMD:R_0603_1608Metric, F.Cu at (80.9, 104.6)
- added R41: R, Resistor_SMD:R_0603_1608Metric, F.Cu at (74.2, 104.6)
- added R42: 100, Resistor_SMD:R_0603_1608Metric, F.Cu at (79.2, 104.6)
- added SW1: SW_Push, Button_Switch_SMD:SW_SPST_CK_RS282G05A3, F.Cu at (196.0, 127.0)
- added SW2: SW_Push, Button_Switch_SMD:SW_SPST_CK_RS282G05A3, F.Cu at (160.0, 129.8)
- added U10: TXS0102DCT, Package_SO:SSOP-8_2.95x2.8mm_P0.65mm, F.Cu at (184.2, 129.8)
- added U6: ATmega328P-A, Package_QFP:TQFP-32_7x7mm_P0.8mm, F.Cu at (189.2, 100.0)
- added U7: FT232RL, Package_SO:SSOP-28_5.3x10.2mm_P0.65mm, F.Cu at (188.2, 118.5)
- added U8: ESP32-WROOM-32, RF_Module:ESP32-WROOM-32, F.Cu at (160.0, 114.5)
- added U9: TXS0102DCT, Package_SO:SSOP-8_2.95x2.8mm_P0.65mm, F.Cu at (157.5, 88.8)
- added Y1: Crystal, Crystal:Crystal_HC49-4H_Vertical, F.Cu at (192.3, 65.0)
- added Y2: Crystal_GND2, Crystal:Resonator_SMD_Murata_CSTxExxV-3Pin_3.0x1.1mm_HandSoldering, F.Cu at (199.2, 97.7)
- C1, C2: value 100nF -> 0.1uF; footprint Capacitor_SMD:C_0402_1005Metric -> Capacitor_SMD:C_0805_2012Metric
- C7, C8: value 0.1uF -> C; footprint Capacitor_SMD:C_0805_2012Metric -> Capacitor_SMD:C_0603_1608Metric
- C9: value 10uF -> C
- D3: value 1N4148W -> D_Filled; footprint Diode_SMD:D_SOD-123 -> Diode_SMD:D_1206_3216Metric_Pad1.42x1.75mm_HandSolder
- H5, H6, H7, H8: footprint MountingHole:MountingHole_4.3mm_M4_DIN965 -> MountingHole:MountingHole_3.2mm_M3
- J1: value Conn_01x07_Female -> Conn_01x02_Male; footprint Connector_PinHeader_2.54mm:PinHeader_1x06_P2.54mm_Vertical -> Connector_Molex:Molex_Micro-Fit_3.0_43650-0200_1x02_P3.00mm_Horizontal
- J2: value Conn_01x03_Female -> Molex Micro-fit 3x1; footprint Connector_PinHeader_2.54mm:PinHeader_1x03_P2.54mm_Vertical -> Connector_Molex:Molex_Micro-Fit_3.0_43650-0300_1x03_P3.00mm_Horizontal
- J4: footprint MountingHole:MountingHole_4.3mm_M4_ISO14580_Pad_TopBottom -> TerminalBlock:TerminalBlock_bornier-2_P5.08mm
- R1, R2, R3, R4: footprint Resistor_SMD:R_1206_3216Metric -> Resistor_SMD:R_0805_2012Metric
- R12: value 0 -> 10k; footprint Resistor_SMD:R_0805_2012Metric -> Resistor_SMD:R_0603_1608Metric
- R13: value 10k -> R; footprint Resistor_SMD:R_0805_2012Metric -> Resistor_SMD:R_0603_1608Metric
- R14: value 0 -> 10k
- R15: value 10k -> 120
- R5, R6: footprint Resistor_SMD:R_0603_1608Metric -> Resistor_SMD:R_0805_2012Metric
- U1: value ESP32_DevKit_V1_DOIT -> LM1117-5; footprint esp32_devkit_v1_doit:esp32_devkit_v1_doit -> Package_TO_SOT_SMD:SOT-223
- U3: value TXS0102DCT -> MCP2515-xSO; footprint Package_SO:SSOP-8_2.95x2.8mm_P0.65mm -> Package_SO:SOIC-18W_7.5x11.6mm_P1.27mm
- U5: value LM1117-5 -> TJA1051T; footprint Package_TO_SOT_SMD:SOT-223 -> Package_SO:SOIC-8_3.9x4.9mm_P1.27mm
- moved C3 186.7 mm to (205.8, 116.3)
- moved R5 169.5 mm to (195.4, 84.5), turned to 90 degrees
- moved C4 164.0 mm to (201.2, 116.3)
- moved U2 161.1 mm to (202.5, 110.8), turned to 90 degrees
- moved C6 151.7 mm to (149.2, 80.8), turned to 180 degrees
- moved R6 148.4 mm to (193.2, 84.5), turned to -90 degrees
- moved R10 145.1 mm to (142.9, 79.0), turned to -90 degrees
- moved H7 144.1 mm to (68.2, 133.5)
- moved C5 141.8 mm to (157.8, 77.0), turned to 90 degrees
- moved R9 140.9 mm to (155.2, 78.0)
- moved R7 138.7 mm to (160.5, 77.0), turned to 90 degrees
- moved J3 137.0 mm to (181.5, 68.2), turned to 0 degrees
- moved U4 134.6 mm to (149.2, 77.8)
- moved R1 134.3 mm to (208.5, 82.0), turned to 90 degrees
- moved H5 128.8 mm to (68.3, 59.5)
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Connections:
- net NANO_3V3 renamed ESP32_VCC
- net Net-(J6-Pad1) renamed /Relay 10A2/NO
- C1 pad 1: GND -> +12V
- C1 pad 2: ESP32_3V3 -> GND
- C2 pad 1: NANO_5V -> GND
- C2 pad 2: GND -> /LM1117 fixed voltage1/VOUT
- C4 pad 2: +5V -> /LM1117 fixed voltage/VOUT
- C7 pad 1: ESP-32_12V -> GND
- C7 pad 2: GND -> Net-(C7-Pad2)
- C8 pad 2: ESP32_VIN -> Net-(C8-Pad2)
- C9 pad 1: NANO_5V -> /CAN Interface/VCC
- D3 pad 2: Net-(D1-Pad1) -> Net-(D3-Pad2)
- F2 pad 1: +5V -> /LM1117 fixed voltage/VOUT
- J1 pad 1: unconnected-(J1-Pad1) -> GND
- J1 pad 2: CAN_SCK -> NANO_D6
- J2 pad 1: CAN_HIGH -> NANO_5V
- J2 pad 2: unconnected-(J2-Pad2) -> GND
- J2 pad 3: CAN_LOW -> ESP32_WS2812B_status_LED_5V
- J3 pad 1: Net-(J3-Pad1) -> /CAN Interface/CAN_H
- J3 pad 2: Net-(J3-Pad2) -> /CAN Interface/CAN_L
- K1 pad 2: Net-(D1-Pad1) -> Net-(D8-Pad1)
- K1 pad 4: unconnected-(K1-Pad4) -> /Relay 10A2/NC
- K2 pad 3: ESP-32_12V -> /Relay 10A/NO
- K2 pad 4: unconnected-(K2-Pad4) -> /Relay 10A/NC
- Q1 pad 1: Net-(Q1-Pad1) -> ESP32_EN_INT
- Q1 pad 3: Net-(D1-Pad1) -> Net-(Q1-Pad3)
- R1 pad 1: ESP-32_SDA_3.3V -> NANO_5V
- R1 pad 2: Net-(R1-Pad2) -> /CAN Interface/VCC
- R12 pad 1: GND -> ESP32_RELAY_1
- R12 pad 2: Net-(R12-Pad2) -> GND
- R13 pad 1: Net-(R12-Pad2) -> NANO_5V
- R13 pad 2: +5V -> Net-(D2-Pad2)
- R14 pad 1: GND -> Net-(R14-Pad1)
- R14 pad 2: Net-(R14-Pad2) -> /CAN Interface/VCC
- R15 pad 1: Net-(R14-Pad2) -> Net-(R15-Pad1)
- R15 pad 2: ESP32_VIN -> Net-(R15-Pad2)
- R16 pad 1: CAN_VCC -> Net-(R15-Pad2)
- R16 pad 2: NANO_5V -> /CAN Interface/CAN_H
- R2 pad 1: ESP-32_SCL_3.3V -> CAN_MOSI
- R3 pad 1: Net-(R3-Pad1) -> CAN_MISO
- R3 pad 2: NANO_SDA_5V -> Net-(R3-Pad2)
- R4 pad 1: Net-(R4-Pad1) -> CAN_CS
- R4 pad 2: NANO_SCL_5V -> Net-(R4-Pad2)
- R5 pad 1: CAN_HIGH -> CAN_SCK
- R5 pad 2: Net-(J3-Pad1) -> Net-(R5-Pad2)
- R6 pad 1: CAN_LOW -> Net-(R6-Pad1)
- R6 pad 2: Net-(J3-Pad2) -> /CAN Interface/INT
- U1 pad 1: unconnected-(U1-Pad1) -> GND
- U1 pad 2: unconnected-(U1-Pad2) -> /LM1117 fixed voltage1/VOUT
- U1 pad 3: unconnected-(U1-Pad3) -> +12V
- U1 pad 4: unconnected-(U1-Pad4) -> (no net)
- U2 pad 1: Net-(R12-Pad2) -> GND
- U2 pad 2: +5V -> /LM1117 fixed voltage/VOUT
- U3 pad 1: Net-(R4-Pad1) -> CAN_TX
- U3 pad 2: GND -> CAN_RX
- U3 pad 3: ESP32_3V3 -> unconnected-(U3-Pad3)
- U3 pad 4: Net-(R2-Pad2) -> unconnected-(U3-Pad4)
- U3 pad 5: Net-(R1-Pad2) -> unconnected-(U3-Pad5)
- U3 pad 7: NANO_5V -> Net-(C7-Pad2)
- U3 pad 8: Net-(R3-Pad1) -> Net-(C8-Pad2)
- U5 pad 1: Net-(R14-Pad2) -> CAN_TX
- U5 pad 2: ESP32_VIN -> GND
- U5 pad 3: ESP-32_12V -> /CAN Interface/VCC
- U5 pad 4: (no net) -> CAN_RX
Routing:
- net NANO_5V: track 0.00 -> 400.7 mm, vias 0 -> 6
- net ESP32_VCC: track 0.00 -> 150.9 mm, vias 0 -> 2
- net +12V: track 0.00 -> 115.4 mm, vias 0 -> 10
- net ESP32_RELAY_4: track 0.00 -> 105.0 mm, vias 0 -> 4
- net ESP32_WS2812B_status_LED_5V: track 0.00 -> 102.2 mm, vias 0 -> 1
- net NANO_D7: track 0.00 -> 87.5 mm, vias 0 -> 2
- net ESP32_RELAY_3: track 0.00 -> 84.5 mm, vias 0 -> 4
- net ESP32_RELAY_2: track 0.00 -> 65.0 mm, vias 0 -> 2
- net ESP32_RELAY_1: track 0.00 -> 64.9 mm, vias 0 -> 4
- net ESP-32_SDA_3.3V: track 0.00 -> 52.8 mm, vias 0 -> 2
- net NANO_RESET: track 0.00 -> 49.3 mm
- net NANO_D6: track 0.00 -> 48.2 mm, vias 0 -> 1
- net ESP-32_SCL_3.3V: track 0.00 -> 46.0 mm
- net Net-(F1-Pad1): track 0.00 -> 42.8 mm
- net Net-(F8-Pad1): track 0.00 -> 39.7 mm
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- added copper zone on B.Cu, net +12V
- added copper zone on F.Cu, net +12V
- added copper zone on F.Cu, net BATTERY
- added copper zone on B.Cu, net GND
- added copper zone on F.Cu, net GND
Other:
- board outline added: 145 x 78 mm
- board text added: "12V"
- board text added: "3.3V LDO"
- board text added: "5.0V LDO"
- board text added: "BATTERY"
- board text added: "CAN_H"
- board text added: "CAN_L"
- board text added: "FLASH"
- board text added: "GND"
- board text added: "GND RX TX 3V3"
- board text added: "Kofferraumbeleuchtung WLED Board"
- board text added: "Kofferraumklappe WLED Board"
- board text added: "VERSORGUNG"
- board text added: "Zigarettenanzünder 1"
- board text added: "Zigarettenanzünder 2"

Commit message: update
Parts:
- added C29: 22uF, Capacitor_SMD:C_0402_1005Metric_Pad0.74x0.62mm_HandSolder, B.Cu at (200.5, 94.5)
- added C30: 100nF, Capacitor_SMD:C_0402_1005Metric_Pad0.74x0.62mm_HandSolder, B.Cu at (192.2, 97.8)
- added C31: 10pF, Capacitor_SMD:C_0805_2012Metric, B.Cu at (199.5, 103.5)
- added C32: 100nF, Capacitor_SMD:C_0402_1005Metric_Pad0.74x0.62mm_HandSolder, B.Cu at (200.8, 106.2)
- added C33: 47uF, Capacitor_SMD:C_1206_3216Metric_Pad1.33x1.80mm_HandSolder, B.Cu at (199.0, 119.0)
- added C34: 47uF, Capacitor_SMD:C_1206_3216Metric_Pad1.33x1.80mm_HandSolder, B.Cu at (199.0, 121.5)
- added D12: B340, Diode_SMD:D_SMC, B.Cu at (188.0, 100.5)
- added J12: Conn_01x02_Male, Connector_Molex:Molex_Micro-Fit_3.0_43650-0200_1x02_P3.00mm_Horizontal, F.Cu at (73.7, 115.5)
- added J13: Conn_01x02_Male, Connector_Molex:Molex_Micro-Fit_3.0_43650-0200_1x02_P3.00mm_Horizontal, F.Cu at (73.7, 126.2)
- added L1: 6.8uH, Inductor_SMD:L_10.4x10.4_H4.8, B.Cu at (191.5, 112.0)
- added R43: 0, Resistor_SMD:R_0603_1608Metric_Pad0.98x0.95mm_HandSolder, B.Cu at (197.5, 92.0)
- added R44: 61.9k, Resistor_SMD:R_0603_1608Metric_Pad0.98x0.95mm_HandSolder, B.Cu at (198.5, 106.2)
- added R45: 10.2k, Resistor_SMD:R_0603_1608Metric_Pad0.98x0.95mm_HandSolder, B.Cu at (198.5, 115.2)
- added R46: 1.96k, Resistor_SMD:R_0603_1608Metric_Pad0.98x0.95mm_HandSolder, B.Cu at (199.5, 112.8)
- C3, C4: value 0.1uF -> 10uF; footprint Capacitor_SMD:C_0805_2012Metric -> Capacitor_SMD:C_1206_3216Metric_Pad1.33x1.80mm_HandSolder; moved to B.Cu
- U2: value LM1117-5 -> TPS54331DDAR; footprint Package_TO_SOT_SMD:SOT-223 -> TPS54331DDAR:CONV_TPS54331DDAR; moved to B.Cu
- U7: value FT232RL -> CH340C; footprint Package_SO:SSOP-28_5.3x10.2mm_P0.65mm -> Package_SO:SOIC-16_3.9x9.9mm_P1.27mm
- moved C3 30.1 mm to (199.2, 87.0)
- moved C4 26.9 mm to (199.2, 89.5)
- moved U2 14.7 mm to (195.8, 97.8), turned to -90 degrees
- moved J5 6.02 mm to (82.8, 128.2)
- moved C18 5.20 mm to (194.2, 114.8)
- moved C1 1.95 mm to (150.8, 131.2)
- moved C2 1.95 mm to (146.2, 131.2)
- moved F3 1.95 mm to (148.8, 135.2)
- moved U1 1.95 mm to (147.5, 125.8)
- moved U7 1.83 mm to (189.8, 119.5), turned to 90 degrees
- moved F1 1.00 mm to (173.5, 78.5)
Connections:
- C1 pad 1: +12V -> +5V
- C4 pad 1: GND -> +12V
- C4 pad 2: /LM1117 fixed voltage/VOUT -> GND
- F2 pad 1: /LM1117 fixed voltage/VOUT -> +5V
- U1 pad 3: +12V -> +5V
- U2 pad 1: GND -> Net-(C30-Pad1)
- U2 pad 2: /LM1117 fixed voltage/VOUT -> +12V
- U2 pad 3: +12V -> Net-(R43-Pad2)
- U2 pad 4: (no net) -> Net-(C29-Pad2)
- U7 pad 1: NANO_TX -> GND
- U7 pad 13: unconnected-(U7-Pad13) -> Net-(C18-Pad1)
- U7 pad 15: Net-(J10-Pad3) -> unconnected-(U7-Pad15)
- U7 pad 16: Net-(J10-Pad2) -> NANO_5V
- U7 pad 2: Net-(C18-Pad1) -> NANO_TX
- U7 pad 3: unconnected-(U7-Pad3) -> NANO_RX
- U7 pad 4: NANO_5V -> unconnected-(U7-Pad4)
- U7 pad 5: NANO_RX -> Net-(J10-Pad3)
- U7 pad 6: unconnected-(U7-Pad6) -> Net-(J10-Pad2)
- U7 pad 7: GND -> unconnected-(U7-Pad7)
- U7 pad 8: (no net) -> unconnected-(U7-Pad8)
- U8 pad 8: /ESP32/GPIO_32 -> ESP_SW1
- U8 pad 9: /ESP32/GPIO_33 -> ESP_SW2
Routing:
- net ESP_SW2: track 0.00 -> 100.5 mm
- net ESP_SW1: track 0.00 -> 93.0 mm
- net +12V: track 115.4 -> 46.3 mm, vias 10 -> 9
- net +5V: track 0.00 -> 67.3 mm, vias 0 -> 2
- net TPS_VSENSE: track 0.00 -> 17.6 mm
- net NANO_RX: track 6.29 -> 23.8 mm
- net NANO_TX: track 5.84 -> 19.9 mm
- net Net-(J10-Pad2): track 25.5 -> 16.6 mm
- net Net-(J10-Pad3): track 26.6 -> 18.0 mm
- net GND: track 35.4 -> 27.0 mm, vias 50 -> 48
- net Net-(C18-Pad1): track 3.73 -> 11.1 mm
- net NANO_RESET: track 49.3 -> 56.3 mm, vias 0 -> 2
- net Net-(C31-Pad2): track 0.00 -> 6.10 mm
- net /LM1117 fixed voltage/VOUT: track 5.97 -> 0.00 mm
- net /CAN Interface/VCC: track 34.2 -> 39.1 mm
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- added copper zone on B.Cu, net +5V
- added copper zone on B.Cu, net /5V 3A Buck/TPS_PH
Other:
- board text added: "RV MAIN PCB Rev.1"

Commit message: assembly V1
Connections:
- C10 pad 1: NANO_5V -> +5V
- C11 pad 1: NANO_5V -> +5V
- C23 pad 1: NANO_5V -> +5V
- C28 pad 1: NANO_5V -> +5V
- D11 pad 1: NANO_5V -> +5V
- D4 pad 1: NANO_5V -> +5V
- D6 pad 1: NANO_5V -> +5V
- D9 pad 1: NANO_5V -> +5V
- K1 pad 5: NANO_5V -> +5V
- K2 pad 5: NANO_5V -> +5V
- K3 pad 5: NANO_5V -> +5V
- K4 pad 5: NANO_5V -> +5V
- R13 pad 1: NANO_5V -> +5V
- R22 pad 1: NANO_5V -> +5V
- R30 pad 1: NANO_5V -> +5V
- R41 pad 1: NANO_5V -> +5V
Routing:
- net +5V: track 67.3 -> 332.4 mm
- net NANO_5V: track 398.8 -> 203.5 mm
Other:
- board text removed: "5.0V LDO"

Commit message: update CAN Frames
Other:
- board text added: "RV MAIN PCB Rev.1.1"
- board text removed: "RV MAIN PCB Rev.1"
Changed lines of the file:
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@@
     (effects (font (size 2 2) (thickness 0.5)))
   )
-  (gr_text "RV MAIN PCB Rev.1" (at 128.75 121.25) (layer "F.SilkS")
+  (gr_text "RV MAIN PCB Rev.1.1\n" (at 128.75 121.25) (layer "F.SilkS")
     (effects (font (size 1.5 1.5) (thickness 0.3)))
   )
